Commit message: make walker.py and fixed urdf

File: urdf/lip_model01.urdf (robot description, URDF)
Before this commit: robot lip01, 5 links, 4 joints
Links:
- link left_foot: mass None -> 0.01
- link left_lowerleg: mass 1e-5 -> 0.1
- link left_upperleg: mass 1e-5 -> 0.1
Joints:
- joint left_knee: limit lower=-0.5 upper=0.5 effort=30 -> lower=-0.5 upper=0.5 effort=10
- joint left_leg_joint: limit lower=-2. upper=2. effort=30 velocity=1.0 -> lower=-2. upper=2. effort=10 velocity=1.0

Commit message: robot get 2 legs and base joint:planar-->floating

File: urdf/lip_model01.urdf (robot description, URDF)
Before this commit: robot lip01, 5 links, 4 joints
Links:
- added link right_foot, mass 0.01; collision sphere radius=0.01; visual sphere radius=0.01
- added link right_lowerleg, mass 0.1; collision cylinder length=0.2 radius=0.01; visual cylinder length=0.2 radius=0.01
- added link right_upperleg, mass 0.1; collision cylinder length=0.2 radius=0.01; visual cylinder length=0.2 radius=0.01
Joints:
- removed joint ankle
- added joint left_ankle: type fixed, parent left_lowerleg, child left_foot, origin xyz=0 0 -0.1 rpy=0 0 0
- added joint right_ankle: type fixed, parent right_lowerleg, child right_foot, origin xyz=0 0 -0.1 rpy=0 0 0
- added joint right_knee: type prismatic, parent right_upperleg, child right_lowerleg, origin xyz=0 0 -0.1 rpy=0 0 0, axis 0 0 1, limit lower=-0.5 upper=0.5 effort=10
- added joint right_leg_joint: type revolute, parent body, child right_upperleg, origin xyz=0 0.05 0 rpy=0 0 0, axis 0 1 0, limit lower=-2. upper=2. effort=10 velocity=1.0
- joint body_joint: type planar -> floating

Commit message: fixed

File: urdf/lip_model01.urdf (robot description, URDF)
Before this commit: robot lip01, 8 links, 7 joints
Links:
- removed link left_foot
- removed link left_lowerleg
- removed link left_upperleg
- removed link right_foot
- removed link right_lowerleg
- removed link right_upperleg
- added link leftFoot, mass 0.01; collision sphere radius=0.01; visual sphere radius=0.01
- added link leftLowerLeg, mass 0.1; collision cylinder length=0.2 radius=0.01; visual cylinder length=0.2 radius=0.01
- added link leftUpperLeg, mass 0.1; collision cylinder length=0.2 radius=0.01; visual cylinder length=0.2 radius=0.01
- added link rightFoot, mass 0.03; collision sphere radius=0.01; visual sphere radius=0.01
- added link rightLowerLeg, mass 0.1; collision cylinder length=0.2 radius=0.01; visual cylinder length=0.2 radius=0.01
- added link rightUpperLeg, mass 0.1; collision cylinder length=0.2 radius=0.01; visual cylinder length=0.2 radius=0.01
Joints:
- removed joint left_ankle
- removed joint left_knee
- removed joint left_leg_joint
- removed joint right_ankle
- removed joint right_knee
- removed joint right_leg_joint
- added joint leftAnkle_joint: type fixed, parent leftLowerLeg, child leftFoot, origin xyz=0 0 -0.2 rpy=0 0 0
- added joint leftHip_joint: type revolute, parent body, child leftUpperLeg, origin xyz=0 -0.05 0 rpy=0 0 0, axis 0 1 0, limit lower=-2. upper=2. effort=10 velocity=1.0
- added joint leftKnee_joint: type revolute, parent leftUpperLeg, child leftLowerLeg, origin xyz=0 0 -0.2 rpy=0 0 0, axis 0 1 0, limit lower=-2 upper=2 effort=10 velocity=1.0
- added joint rightAnkle: type fixed, parent rightLowerLeg, child rightFoot, origin xyz=0 0 -0.2 rpy=0 0 0
- added joint rightHip_joint: type revolute, parent body, child rightUpperLeg, origin xyz=0 0.05 0 rpy=0 0 0, axis 0 1 0, limit lower=-2. upper=2. effort=10 velocity=1.0
- added joint rightKnee_joint: type revolute, parent rightUpperLeg, child rightLowerLeg, origin xyz=0 0 -0.2 rpy=0 0 0, axis 0 1 0, limit lower=-2. upper=2. effort=10 velocity=1.0
- joint body_joint: axis 1 0 1 -> (none); type floating -> fixed

Commit message: update

File: urdf/lip_model01.urdf (robot description, URDF)
Before this commit: robot lip01, 8 links, 7 joints
Links:
- link leftFoot: geometry collision box size=0.02 0.1 0.01; visual box size=0.02 0.1 0.01
- link rightFoot: geometry collision box size=0.02 0.1 0.01; visual box size=0.02 0.1 0.01
Joints:
- joint leftAnkle_joint: axis (none) -> 0 1 0; limit (none) -> lower=-2. upper=2 effort=1. velocity=10.; type fixed -> revolute
- joint leftHip_joint: limit lower=-2. upper=2. effort=10 velocity=1.0 -> lower=-2. upper=2. effort=10. velocity=1.0
- joint leftKnee_joint: limit lower=-2 upper=2 effort=10 velocity=1.0 -> lower=-2. upper=2. effort=10. velocity=1.0
- joint rightAnkle: axis (none) -> 0 1 0; limit (none) -> lower=-2. upper=2. effort=1. velocity=10.; type fixed -> revolute
- joint rightHip_joint: limit lower=-2. upper=2. effort=10 velocity=1.0 -> lower=-2. upper=2. effort=10. velocity=1.0
- joint rightKnee_joint: limit lower=-2. upper=2. effort=10 velocity=1.0 -> lower=-2. upper=2. effort=10. velocity=1.0

Commit message: add generateLIPWalkingPattern.py

File: urdf/lip_model01.urdf (robot description, URDF)
Before this commit: robot lip01, 8 links, 7 joints
Links:
- removed link base
- added link world
Joints:
- joint body_joint: parent base -> world

Commit message: update

File: urdf/lip_model01.urdf (robot description, URDF)
Before this commit: robot lip01, 8 links, 7 joints
Links:
- removed link world
- added link base
- link leftFoot: geometry collision box size=0.04 0.1 0.01; visual box size=0.02 0.1 0.01
- link rightFoot: geometry collision box size=0.04 0.1 0.01; visual box size=0.02 0.1 0.01
Joints:
- removed joint rightAnkle
- added joint rightAnkle_joint: type revolute, parent rightLowerLeg, child rightFoot, origin xyz=0 0 -0.2 rpy=0 0 0, axis 0 -1 0, limit lower=-2. upper=2. effort=1. velocity=10.
- joint body_joint: parent world -> base
- joint rightHip_joint: axis 0 1 0 -> 0 -1 0
- joint rightKnee_joint: axis 0 1 0 -> 0 -1 0
